File: Spi_Flash_Development_Board.kicad_pcb (KiCad board)
At the start: 2 copper layers, 91.8 x 60 mm, 44 parts, among them P1 BPi_Main_Interface, P2 ~CS~_Common, P3 ~CS~_Common, P4 ~CS~_Common, P5 ~CS~_Common, P6 ~CS~_Common, P7 ~CS~_Common, P8 BPi-4Pin_Interface, P9 BPi-2Pin_Interface, Sw1 D6R_SPST_MKS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

Commit message: RC1 of Banana Pi Flash Memory Interface
Parts:
- moved D3 149.8 mm to (190.9, 88.0), turned to 90 degrees
- moved C4 139.4 mm to (189.1, 88.0), turned to 90 degrees
- moved D6 137.5 mm to (174.1, 114.2), turned to 180 degrees
- moved C6 136.0 mm to (186.4, 88.2)
- moved C5 129.3 mm to (178.5, 92.2), turned to 90 degrees
- moved U5 128.8 mm to (173.5, 106.9)
- moved R5 128.0 mm to (183.8, 88.4), turned to 90 degrees
- moved R3 126.8 mm to (164.4, 94.1), turned to 180 degrees
- moved R6 124.2 mm to (171.4, 113.2), turned to 90 degrees
- moved D2 121.4 mm to (163.4, 96.7), turned to 90 degrees
- moved U7 121.1 mm to (171.0, 92.2), turned to 270 degrees
- moved D4 120.7 mm to (162.6, 114.2), turned to 180 degrees
- moved D1 120.6 mm to (151.2, 114.2), turned to 180 degrees
- moved C11 116.3 mm to (176.7, 92.2), turned to 90 degrees
- moved R4 116.1 mm to (159.9, 113.2), turned to 90 degrees
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Connections:
- D1 pad 1: GND -> 3V3
- D4 pad 1: GND -> 3V3
- D5 pad 1: GND -> 3V3
- D6 pad 1: GND -> 3V3
- P1 pad 10: ~SIG_BUSY -> ~SIG_CS1
- P1 pad 11: ~SIG_CS -> SIG_SIO3
- P1 pad 13: SIG_SIO1 -> SIG_SIO2
- P1 pad 15: SIG_SIO2 -> SIG_SIO1
- P1 pad 16: SIG_SIO3 -> SIG_DIR_IO
- P1 pad 18: SIG_SCK -> ~SIG_CS6
- P1 pad 19: ~SIG_CS2 -> ~SIG_RST
- P1 pad 21: ~SIG_CS3 -> ~SIG_WP
- P1 pad 22: SIG_DIR_IO -> SIG_SCK
- P1 pad 23: ~SIG_CS4 -> SIG_BTN
- P1 pad 26: ~SIG_CS6 -> ~SIG_BUSY
- P1 pad 3: ~SIG_RST -> ~SIG_CS3
- P1 pad 5: ~SIG_WP -> ~SIG_CS4
- P8 pad 3: ~SIG_CS1 -> ~SIG_CS
- P8 pad 5: SIG_BTN -> ~SIG_CS2
- U1 pad 16: SIG_BUF_SIO2 -> SIG_BUF_SIO0
- U1 pad 17: SIG_BUF_SIO1 -> SIG_BUF_SIO2
- U1 pad 18: SIG_BUF_SIO0 -> SIG_BUF_SIO1
- U1 pad 2: SIG_SIO0 -> SIG_SIO1
- U1 pad 3: SIG_SIO1 -> SIG_SIO2
- U1 pad 4: SIG_SIO2 -> SIG_SIO0
- U6 pad 13: SIG_BUF_SIO0 -> SIG_SIO0
- U7 pad 1: SIG_BUF_SIO0 -> SIG_SIO0
Routing:
- net GND: track 0.00 -> 300.4 mm, vias 0 -> 16
- net 3V3: track 0.00 -> 246.8 mm, vias 0 -> 3
- net SIG_BUF_SIO1: track 0.00 -> 121.3 mm
- net ~SIG_CS: track 0.00 -> 107.7 mm
- net SIG_SCK: track 0.00 -> 107.6 mm, vias 0 -> 3
- net ~SIG_CS4: track 0.00 -> 86.4 mm, vias 0 -> 2
- net ~SIG_CS3: track 0.00 -> 76.6 mm, vias 0 -> 2
- net SIG_BUF_SIO2: track 0.00 -> 75.9 mm
- net SIG_BUF_SIO0: track 0.00 -> 71.7 mm
- net SIG_BUF_SIO3: track 0.00 -> 64.8 mm
- net ~SIG_RST: track 0.00 -> 63.9 mm, vias 0 -> 2
- net SIG_SIO0: track 0.00 -> 60.0 mm
- net ~SIG_WP: track 0.00 -> 59.9 mm, vias 0 -> 2
- net ~SIG_CS6: track 0.00 -> 52.3 mm, vias 0 -> 2
- net ~SIG_CS2: track 0.00 -> 50.3 mm
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- added copper zone on B.Cu, net GND
- added copper zone on F.Cu, net GND
Other:
- net class Default: trace_width 0.25 -> 0.254; via_dia 0.6 -> 1; via_drill 0.4 -> 0.6
- board text added: "Banana Pi Flash Memory Interface"
- board text added: "Revision V1_0"

Commit message: Final verion of board V1_0. Prototype started.
Connections:
- P8 pad 6: Net-(P8-Pad6) -> SIG_LED
- P9 pad 1: SIG_LED -> Net-(P9-Pad1)
Routing:
- net GND: track 300.4 -> 389.7 mm, vias 16 -> 19
- net SIG_LED: track 32.4 -> 35.7 mm
- net 3V3: track 246.8 -> 248.1 mm
Other:
- outline, holes or cut-outs redrawn
- board text added: "Banana Pi Flash Memory Interface Revision V1_0"
- board text added: "Banana Pi pins description(Wiring Pi): CS-GPIO17,CS1-GPIO16,CS2-GPIO19,CS3-GPIO8, CS4-GPIO9,CS5-GPIO10,CS6-GPIO5,LED-GPIO20 BUTTON-GPIO14,RESET-GPIO12,WP-GPIO13, SCLK-GPIO6,DIR-GPIO4,MOSI-GPIO1,MISO-GPIO3 SIO0-GPIO1,SIO1-GPIO3,SIO2-GPIO2,SIO3-GPIO0"
- board text added: "VOLOVIQUE 2017"
- board text removed: "Banana Pi Flash Memory Interface"
- board text removed: "Revision V1_0"
