File: Spi_Flash_Development_Board.sch (KiCad schematic (older format))
At the start: 44 parts, among them P1 BPi_Main_Interface, P2 ~CS~_Common, P3 ~CS~_Common, P4 ~CS~_Common, P5 ~CS~_Common, P6 ~CS~_Common, P7 ~CS~_Common, P8 BPi-4Pin_Interface, P9 BPi-2Pin_Interface, Sw1 D6R_SPST_MKS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

Commit message: RC1 of Banana Pi Flash Memory Interface
Connections:
- net 3V3: now also D1.1 (A), D4.1 (A), D5.1 (A), D6.1 (A)
- net GND: no longer D1.1 (A), D4.1 (A), D5.1 (A), D6.1 (A)
- net SIG_BTN: now also P1.23; no longer P8.5
- net SIG_BUF_SIO0: now also U1.16 (B2); no longer U1.18 (B0), U6.13 (SI), U7.1 (SI)
- net SIG_BUF_SIO1: now also U1.18 (B0); no longer U1.17 (B1)
- net SIG_BUF_SIO2: now also U1.17 (B1); no longer U1.16 (B2)
- net SIG_DIR_IO: now also P1.16; no longer P1.22
- net SIG_SCK: now also P1.22; no longer P1.18
- net SIG_SIO0: now also U1.4 (A2), U6.13 (SI), U7.1 (SI); no longer U1.2 (A0)
- net SIG_SIO1: now also P1.15, U1.2 (A0); no longer P1.13, U1.3 (A1)
- net SIG_SIO2: now also P1.13, U1.3 (A1); no longer P1.15, U1.4 (A2)
- net SIG_SIO3: now also P1.11; no longer P1.16
- net ~SIG_BUSY: now also P1.26; no longer P1.10
- net ~SIG_CS: now also P8.3; no longer P1.11
- net ~SIG_CS1: now also P1.10; no longer P8.3
- net ~SIG_CS2: now also P8.5; no longer P1.19
- net ~SIG_CS3: now also P1.3; no longer P1.21
- net ~SIG_CS4: now also P1.5; no longer P1.23
- net ~SIG_CS6: now also P1.18; no longer P1.26
- net ~SIG_RST: now also P1.19; no longer P1.3
- net ~SIG_WP: now also P1.21; no longer P1.5

Commit message: Final verion of board V1_0. Prototype started.
Connections:
- net SIG_LED: now also P8.6; no longer P9.1
Other:
- note added: "GPIO0"
- note added: "GPIO1"
- note added: "GPIO10"
- note added: "GPIO11"
- note added: "GPIO12"
- note added: "GPIO13"
- note added: "GPIO14"
- note added: "GPIO15"
- note added: "GPIO16"
- note added: "GPIO17"
- note added: "GPIO18"
- note added: "GPIO19"
- note added: "GPIO2"
- note added: "GPIO20"
- note added: "GPIO3"
- note added: "GPIO4"
- note added: "GPIO5"
- note added: "GPIO6"
- note added: "GPIO7"
- note added: "GPIO8"
- note added: "GPIO9"
Changed lines of the file:
@@
 NoConn ~ 1450 5200
 NoConn ~ 2250 6650
-NoConn ~ 2250 6750
 NoConn ~ 1500 7450
 NoConn ~ 1450 6550
@@
 	-1   0    0    1
 $EndComp
-Text GLabel 1350 7350 0    39   Output ~ 0
+Text GLabel 2250 6750 2    39   Output ~ 0
 SIG_LED
-Wire Wire Line
-	1500 7350 1350 7350
 $Comp
 L 330R_0805 R8
@@
 	3450 2750 3450 3050
 Connection ~ 3450 3050
+Text Notes 700  5050 0    60   ~ 0
+GPIO8
+Text Notes 700  5150 0    60   ~ 0
+GPIO9
+Text Notes 700  5450 0    60   ~ 0
+GPIO0
+Text Notes 700  5550 0    60   ~ 0
+GPIO2
+Text Notes 700  5650 0    60   ~ 0
+GPIO3
+Text Notes 700  5850 0    60   ~ 0
+GPIO12
+Text Notes 700  5950 0    60   ~ 0
+GPIO13
+Text Notes 700  6050 0    60   ~ 0
+GPIO14
+Text Notes 2750 6150 0    60   ~ 0
+GPIO11
+Text Notes 2750 6050 0    60   ~ 0
+GPIO10
+Text Notes 2750 5950 0    60   ~ 0
+GPIO6
+Text Notes 2750 5750 0    60   ~ 0
+GPIO5
+Text Notes 2750 5650 0    60   ~ 0
+GPIO4
+Text Notes 2750 5450 0    60   ~ 0
+GPIO1
+Text Notes 2750 5350 0    60   ~ 0
+GPIO16
+Text Notes 700  6700 0    60   ~ 0
+GPIO17
+Text Notes 2600 6700 0    60   ~ 0
+GPIO18
+Text Notes 700  6800 0    60   ~ 0
+GPIO19
+Text Notes 2600 6800 0    60   ~ 0
+GPIO20
+NoConn ~ 1500 7350
+Text Notes 700  5250 0    60   ~ 0
+GPIO7
+Text Notes 2750 5250 0    60   ~ 0
+GPIO15
 $EndSCHEMATC
